Commit message: edit local costmap param

File: src/gz_bringup/urdf/x1_robot.urdf (robot description, URDF)
Before this commit: robot x1_robot, 3 links, 2 joints
Joints:
- joint lidar_joint: origin xyz=0.0 0.0 0.4 rpy=0 0 0 -> xyz=0.5 0.0 0.2 rpy=0 0 0

Commit message: Add dual lidar

File: src/gz_bringup/urdf/x1_robot.urdf (robot description, URDF)
Before this commit: robot x1_robot, 3 links, 2 joints
Links:
- added link lidar_rear_link; visual cylinder length=0.08 radius=0.06
Joints:
- added joint lidar_rear_joint: type fixed, parent base_link, child lidar_rear_link, origin xyz=-0.5 0.0 0.2 rpy=0 0 3.14159
